Commit message: Collected data a

File: assets/pybullet/orange_cup/model.urdf (robot description, URDF)
Before this commit: robot model.urdf, 1 links, 0 joints
Links:
- link baseLink: geometry collision mesh filename=collision.obj scale=0.9 0.9 0.9; visual mesh filename=textured.obj scale=0.9 0.9 0.9
